File: boards/LaserCardV2/boardv1.brd (EAGLE design)
At the start: 100 x 69.8 mm, 30 parts, among them K1 NA, K3 NA, K4 NA, K6 NA, X1 112404, X2 112404, X3 112404, X4 112404, X5 112404, X6 112404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

Commit message: Board update
Parts:
- added R2: 0, SparkFun-Resistors:0603
- C2: device SparkFun-Capacitors:CAP-PTH-SMALL-KIT -> SparkFun-Capacitors:0603-CAP
- moved JP4 53.4 mm to (41.9, 22.9)
- moved R9 49.4 mm to (19.1, 50.8), turned to 180 degrees
- moved D1 49.0 mm to (14.0, 52.7), turned to 270 degrees
- moved D5 49.0 mm to (33.0, 52.7), turned to 270 degrees
- moved R5 49.0 mm to (38.1, 50.8), turned to 180 degrees
- moved D12 49.0 mm to (71.1, 52.7), turned to 270 degrees
- moved D7 49.0 mm to (52.1, 52.7), turned to 270 degrees
- moved R1 48.7 mm to (57.1, 50.8), turned to 180 degrees
- moved R12 48.7 mm to (76.2, 50.8), turned to 180 degrees
- moved JP1 48.0 mm to (97.2, 59.1), turned to 90 degrees
- moved X5 46.8 mm to (57.1, 24.8)
- moved JP2 43.0 mm to (97.2, 48.9), turned to 270 degrees
- moved D8 41.3 mm to (57.1, 48.3)
- moved C2 38.9 mm to (81.3, 59.1)
- moved D2 35.8 mm to (19.1, 48.3), turned to 0 degrees
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Connections:
- new net GND2: C1.2, C2.2, IC1.9, JP1.1, R2.2
- net GND: now also R2.1; no longer C1.2, C2.2, IC1.9, JP1.1
- net R1: now also D11.A, K6.12, R12.1
- net R2: now also D8.A, K4.12, R1.1; no longer D11.A, K6.12, R12.1
- net R3: now also D6.A, K3.12, R5.1
- net R4: now also D2.A, K1.12, R9.1; no longer D8.A, K4.12, R1.1
- net R5: no longer D6.A, K3.12, R5.1
- net R6: no longer D2.A, K1.12, R9.1
Routing:
- net R6: track 127.9 -> 0.00 mm, vias 5 -> 0
- net R5: track 85.5 -> 0.00 mm, vias 2 -> 0
- net N$1: track 112.5 -> 39.0 mm, vias 4 -> 2
- net R3: track 0.00 -> 71.8 mm, vias 0 -> 2
- net ARDUINO1: track 106.7 -> 46.7 mm
- net GND2: track 0.00 -> 48.9 mm, vias 0 -> 1
- net OUTPUT1: track 66.4 -> 30.5 mm
- net R4: track 58.7 -> 91.8 mm
- net GND: track 29.7 -> 0.00 mm, vias 0 -> 3
- net SIG4A: track 15.5 -> 45.2 mm, vias 0 -> 2
- net OUTPUTA: track 60.5 -> 31.5 mm, vias 2 -> 0
- net R1: track 0.00 -> 21.2 mm, vias 0 -> 1
- net OUTPUT2: track 39.1 -> 18.0 mm
- net OUTPUT4: track 25.1 -> 41.6 mm
- net O2: track 41.7 -> 53.3 mm
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- added copper zone on layer 1, net GND
- added copper zone on layer 16, net GND2
Other:
- board text added: "1A"
- board text added: "1D"
- board text added: "2A"
- board text added: "2D"
- board text added: "MON"
- board text removed: "420A"
- board text removed: "420D"
- board text removed: "660A"
- board text removed: "660D"
- board text removed: "BYPASS"
