File: boards/LaserCardV2/boardv1.sch (EAGLE design)
At the start: 30 parts, among them K1 NA, K3 NA, K4 NA, K6 NA, X1 112404, X2 112404, X3 112404, X4 112404, X5 112404, X6 112404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

Commit message: Board update
Parts:
- added R2: 0, SparkFun-Resistors:0OHM-1/10W-5%(0603)
- C2: device SparkFun-Capacitors:0.1UF-50V-20%(PTH)KIT-EZ -> SparkFun-Capacitors:0.1UF-25V-5%(0603)
Connections:
- new net GND2: C1.-, C2.2, IC1.GND, JP1.1, R2.2
- net GND: now also R2.1; no longer C1.-, C2.2, IC1.GND, JP1.1
- net R1: now also D11.A, K61.-, R12.1
- net R2: now also D8.A, K41.-, R1.1; no longer D11.A, K61.-, R12.1
- net R3: now also D6.A, K31.-, R5.1
- net R4: now also D2.A, K11.-, R9.1; no longer D8.A, K41.-, R1.1
- net R5: no longer D6.A, K31.-, R5.1
- net R6: no longer D2.A, K11.-, R9.1
